File: pcbs/slave_drum.sch (KiCad schematic (older format))
At the start: 22 parts, among them J1 Screw_Terminal_01x02, J2 Conn_02x04_Odd_Even, U1 LF15_TO220

Commit message: finished slave pcb
Parts:
- added D6: D, Diodes_THT:D_DO-201AD_P12.70mm_Horizontal, symbol D
- C1: renamed from C?; footprint (none) -> Capacitors_THT:CP_Radial_D4.0mm_P2.00mm
- D1, D2, D4, D5: renamed from D?; footprint (none) -> LEDs:LED-5MM
- D3: renamed from D?; footprint (none) -> Diodes_THT:D_DO-201_P12.70mm_Horizontal
- J3, J4: renamed from J?; footprint (none) -> Pin_Headers:Pin_Header_Straight_1x02
- JP1, JP2: renamed from JP?; footprint (none) -> jumper:SOLDER-JUMPER_1-WAY_FAR
- R1, R2, R3, R4, R5, R6: renamed from R?; footprint (none) -> Resistors_THT:R_Axial_DIN0207_L6.3mm_D2.5mm_P7.62mm_Horizontal
- U1: footprint Power_Integrations:TO-220 -> TO_SOT_Packages_THT:TO-220_Horizontal
- uP1: footprint (none) -> ArduProMiniTKB:ArduProMini-6
- gave numbers to parts that had none: 2
Connections:
- net +12V: now also U1.1 (VI), D6.1 (K)
- net +12C: no longer names the net of J1.2 (Pin_2)
- net +12C: now also D6.2 (A); no longer U1.1 (VI)
- net Earth renamed GND
Other:
- moved on the sheet: J1

Commit message: added bom
Parts:
- C1: footprint Capacitors_THT:CP_Radial_D4.0mm_P2.00mm -> Capacitors_THT:CP_Radial_D5.0mm_P2.00mm
Changed lines of the file:
@@
 F 0 "C1" H 6075 1450 50  0000 L CNN
 F 1 "CP" H 6075 1250 50  0000 L CNN
-F 2 "Capacitors_THT:CP_Radial_D4.0mm_P2.00mm" H 6088 1200 50  0001 C CNN
+F 2 "Capacitors_THT:CP_Radial_D5.0mm_P2.00mm" H 6088 1200 50  0001 C CNN
 F 3 "" H 6050 1350 50  0001 C CNN
 F 4 "10 uF" H 6050 1350 60  0000 C TNN "Capacitance"
